File: kicad/mp3_player/max98357.kicad_sch (KiCad schematic)
At the start: 8 parts, among them U6 MAX98357A

Commit message: [FIX] the schematic tracking issue in KiCad
Parts:
- renumbered C7 to C15, C8 to C16, C9 to C17, C10 to C18, L1 to L5, L2 to L6, R16 to R18, U6 to U8
Changed lines of the file:
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@@
 		(dnp no)
 		(fields_autoplaced yes)
-		(property "Reference" "U6"
+		(property "Reference" "U8"
 			(at 54.2133 26.67 0)
 			(show_name no)
@@
 					(unit 1)
 				)
-				(path "/0f0043d3-9467-400d-886a-57a73f910f34/a50beffe-a239-4916-9845-73f6497a511a"
-					(reference "U6")
+				(path "/0f0043d3-9467-400d-886a-57a73f910f34/cfa83fee-df6a-42e6-9021-3f2792ba73ef"
+					(reference "U8")
 					(unit 1)
 				)
@@
 		(dnp no)
 		(fields_autoplaced yes)
-		(property "Reference" "C9"
+		(property "Reference" "C17"
 			(at 77.47 44.4562 0)
 			(show_name no)
@@
 					(unit 1)
 				)
-				(path "/0f0043d3-9467-400d-886a-57a73f910f34/a50beffe-a239-4916-9845-73f6497a511a"
-					(reference "C9")
+				(path "/0f0043d3-9467-400d-886a-57a73f910f34/cfa83fee-df6a-42e6-9021-3f2792ba73ef"
+					(reference "C17")
 					(unit 1)
 				)
@@
 		(dnp no)
 		(fields_autoplaced yes)
-		(property "Reference" "C8"
+		(property "Reference" "C16"
 			(at 45.72 21.5962 0)
 			(show_name no)
@@
 					(unit 1)
 				)
-				(path "/0f0043d3-9467-400d-886a-57a73f910f34/a50beffe-a239-4916-9845-73f6497a511a"
-					(reference "C8")
+				(path "/0f0043d3-9467-400d-886a-57a73f910f34/cfa83fee-df6a-42e6-9021-3f2792ba73ef"
+					(reference "C16")
 					(unit 1)
 				)
@@
 		(dnp no)
 		(fields_autoplaced yes)
-		(property "Reference" "#PWR025"
+		(property "Reference" "#PWR038"
 			(at 43.18 15.24 0)
 			(hide yes)
@@
 					(unit 1)
 				)
-				(path "/0f0043d3-9467-400d-886a-57a73f910f34/a50beffe-a239-4916-9845-73f6497a511a"
-					(reference "#PWR025")
+				(path "/0f0043d3-9467-400d-886a-57a73f910f34/cfa83fee-df6a-42e6-9021-3f2792ba73ef"
+					(reference "#PWR038")
 					(unit 1)
 				)
@@
 		(dnp no)
 		(fields_autoplaced yes)
-		(property "Reference" "C10"
+		(property "Reference" "C18"
 			(at 88.9 44.4562 0)
 			(show_name no)
@@
 					(unit 1)
 				)
-				(path "/0f0043d3-9467-400d-886a-57a73f910f34/a50beffe-a239-4916-9845-73f6497a511a"
-					(reference "C10")
+				(path "/0f0043d3-9467-400d-886a-57a73f910f34/cfa83fee-df6a-42e6-9021-3f2792ba73ef"
+					(reference "C18")
 					(unit 1)
 				)
@@
 		(dnp no)
 		(fields_autoplaced yes)
-		(property "Reference" "#PWR024"
+		(property "Reference" "#PWR037"
 			(at 34.29 15.24 0)
 			(hide yes)
@@
 					(unit 1)
 				)
-				(path "/0f0043d3-9467-400d-886a-57a73f910f34/a50beffe-a239-4916-9845-73f6497a511a"
-					(reference "#PWR024")
+				(path "/0f0043d3-9467-400d-886a-57a73f910f34/cfa83fee-df6a-42e6-9021-3f2792ba73ef"
+					(reference "#PWR037")
 					(unit 1)
 				)
@@
 		(in_pos_files yes)
 		(dnp no)
-		(property "Reference" "L2"
+		(property "Reference" "L6"
 			(at 80.01 30.226 0)
 			(show_name no)
@@
 					(unit 1)
 				)
-				(path "/0f0043d3-9467-400d-886a-57a73f910f34/a50beffe-a239-4916-9845-73f6497a511a"
-					(reference "L2")
+				(path "/0f0043d3-9467-400d-886a-57a73f910f34/cfa83fee-df6a-42e6-9021-3f2792ba73ef"
+					(reference "L6")
 					(unit 1)
 				)
@@
 		(dnp no)
 		(fields_autoplaced yes)
-		(property "Reference" "#PWR028"
+		(property "Reference" "#PWR041"
 			(at 74.93 62.23 0)
 			(hide yes)
@@
 					(unit 1)
 				)
-				(path "/0f0043d3-9467-400d-886a-57a73f910f34/a50beffe-a239-4916-9845-73f6497a511a"
-					(reference "#PWR028")
+				(path "/0f0043d3-9467-400d-886a-57a73f910f34/cfa83fee-df6a-42e6-9021-3f2792ba73ef"
+					(reference "#PWR041")
 					(unit 1)
 				)
@@
 		(dnp no)
 		(fields_autoplaced yes)
-		(property "Reference" "L1"
+		(property "Reference" "L5"
 			(at 69.85 26.67 0)
 			(show_name no)
@@
 					(unit 1)
 				)
-				(path "/0f0043d3-9467-400d-886a-57a73f910f34/a50beffe-a239-4916-9845-73f6497a511a"
-					(reference "L1")
+				(path "/0f0043d3-9467-400d-886a-57a73f910f34/cfa83fee-df6a-42e6-9021-3f2792ba73ef"
+					(reference "L5")
 					(unit 1)
 				)
@@
 		(dnp no)
 		(fields_autoplaced yes)
-		(property "Reference" "#PWR026"
+		(property "Reference" "#PWR039"
 			(at 49.53 62.23 0)
 			(hide yes)
@@
 					(unit 1)
 				)
-				(path "/0f0043d3-9467-400d-886a-57a73f910f34/a50beffe-a239-4916-9845-73f6497a511a"
-					(reference "#PWR026")
+				(path "/0f0043d3-9467-400d-886a-57a73f910f34/cfa83fee-df6a-42e6-9021-3f2792ba73ef"
+					(reference "#PWR039")
 					(unit 1)
 				)
@@
 		(dnp no)
 		(fields_autoplaced yes)
-		(property "Reference" "#PWR029"
+		(property "Reference" "#PWR042"
 			(at 86.36 62.23 0)
 			(hide yes)
@@
 					(unit 1)
 				)
-				(path "/0f0043d3-9467-400d-886a-57a73f910f34/a50beffe-a239-4916-9845-73f6497a511a"
-					(reference "#PWR029")
+				(path "/0f0043d3-9467-400d-886a-57a73f910f34/cfa83fee-df6a-42e6-9021-3f2792ba73ef"
+					(reference "#PWR042")
 					(unit 1)
 				)
@@
 		(dnp no)
 		(fields_autoplaced yes)
-		(property "Reference" "C7"
+		(property "Reference" "C15"
 			(at 36.83 21.5962 0)
 			(show_name no)
@@
 					(unit 1)
 				)
-				(path "/0f0043d3-9467-400d-886a-57a73f910f34/a50beffe-a239-4916-9845-73f6497a511a"
-					(reference "C7")
+				(path "/0f0043d3-9467-400d-886a-57a73f910f34/cfa83fee-df6a-42e6-9021-3f2792ba73ef"
+					(reference "C15")
 					(unit 1)
 				)
@@
 		(dnp no)
 		(fields_autoplaced yes)
-		(property "Reference" "#PWR027"
+		(property "Reference" "#PWR040"
 			(at 54.61 62.23 0)
 			(hide yes)
@@
 					(unit 1)
 				)
-				(path "/0f0043d3-9467-400d-886a-57a73f910f34/a50beffe-a239-4916-9845-73f6497a511a"
-					(reference "#PWR027")
+				(path "/0f0043d3-9467-400d-886a-57a73f910f34/cfa83fee-df6a-42e6-9021-3f2792ba73ef"
+					(reference "#PWR040")
 					(unit 1)
 				)
@@
 		(in_pos_files yes)
 		(dnp no)
-		(property "Reference" "R16"
+		(property "Reference" "R18"
 			(at 24.13 38.354 90)
 			(show_name no)
@@
 					(unit 1)
 				)
-				(path "/0f0043d3-9467-400d-886a-57a73f910f34/a50beffe-a239-4916-9845-73f6497a511a"
-					(reference "R16")
-					(unit 1)
-				)
+				(path "/0f0043d3-9467-400d-886a-57a73f910f34/cfa83fee-df6a-42e6-9021-3f2792ba73ef"
+					(reference "R18")
+					(unit 1)
+				)

Commit message: [ADD] lcd segment displays to the project
Parts:
- renumbered C18 to C10, C15 to C7, C16 to C8, C17 to C9, L5 to L1, L6 to L2, R18 to R16, U8 to U6
Changed lines of the file:
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@@
 		(dnp no)
 		(fields_autoplaced yes)
-		(property "Reference" "U8"
+		(property "Reference" "U6"
 			(at 54.2133 26.67 0)
 			(show_name no)
@@
 				)
 				(path "/0f0043d3-9467-400d-886a-57a73f910f34/cfa83fee-df6a-42e6-9021-3f2792ba73ef"
-					(reference "U8")
+					(reference "U6")
 					(unit 1)
 				)
@@
 		(dnp no)
 		(fields_autoplaced yes)
-		(property "Reference" "C17"
+		(property "Reference" "C9"
 			(at 77.47 44.4562 0)
 			(show_name no)
@@
 				)
 				(path "/0f0043d3-9467-400d-886a-57a73f910f34/cfa83fee-df6a-42e6-9021-3f2792ba73ef"
-					(reference "C17")
+					(reference "C9")
 					(unit 1)
 				)
@@
 		(dnp no)
 		(fields_autoplaced yes)
-		(property "Reference" "C16"
+		(property "Reference" "C8"
 			(at 45.72 21.5962 0)
 			(show_name no)
@@
 				)
 				(path "/0f0043d3-9467-400d-886a-57a73f910f34/cfa83fee-df6a-42e6-9021-3f2792ba73ef"
-					(reference "C16")
+					(reference "C8")
 					(unit 1)
 				)
@@
 		(dnp no)
 		(fields_autoplaced yes)
-		(property "Reference" "#PWR038"
+		(property "Reference" "#PWR028"
 			(at 43.18 15.24 0)
 			(hide yes)
@@
 			(project "mp3_player"
 				(path "/0f0043d3-9467-400d-886a-57a73f910f34/4f719e08-a5fd-46cb-a375-4f681db4c0e1"
-					(reference "#PWR031")
+					(reference "#PWR034")
 					(unit 1)
 				)
 				(path "/0f0043d3-9467-400d-886a-57a73f910f34/cfa83fee-df6a-42e6-9021-3f2792ba73ef"
-					(reference "#PWR038")
+					(reference "#PWR028")
 					(unit 1)
 				)
@@
 		(dnp no)
 		(fields_autoplaced yes)
-		(property "Reference" "C18"
+		(property "Reference" "C10"
 			(at 88.9 44.4562 0)
 			(show_name no)
@@
 				)
 				(path "/0f0043d3-9467-400d-886a-57a73f910f34/cfa83fee-df6a-42e6-9021-3f2792ba73ef"
-					(reference "C18")
+					(reference "C10")
 					(unit 1)
 				)
@@
 		(dnp no)
 		(fields_autoplaced yes)
-		(property "Reference" "#PWR037"
+		(property "Reference" "#PWR027"
 			(at 34.29 15.24 0)
 			(hide yes)
@@
 			(project "mp3_player"
 				(path "/0f0043d3-9467-400d-886a-57a73f910f34/4f719e08-a5fd-46cb-a375-4f681db4c0e1"
-					(reference "#PWR030")
+					(reference "#PWR033")
 					(unit 1)
 				)
 				(path "/0f0043d3-9467-400d-886a-57a73f910f34/cfa83fee-df6a-42e6-9021-3f2792ba73ef"
-					(reference "#PWR037")
+					(reference "#PWR027")
 					(unit 1)
 				)
@@
 		(in_pos_files yes)
 		(dnp no)
-		(property "Reference" "L6"
+		(property "Reference" "L2"
 			(at 80.01 30.226 0)
 			(show_name no)
@@
 				)
 				(path "/0f0043d3-9467-400d-886a-57a73f910f34/cfa83fee-df6a-42e6-9021-3f2792ba73ef"
-					(reference "L6")
+					(reference "L2")
 					(unit 1)
 				)
@@
 		(dnp no)
 		(fields_autoplaced yes)
-		(property "Reference" "#PWR041"
+		(property "Reference" "#PWR031"
 			(at 74.93 62.23 0)
 			(hide yes)
@@
 			(project "mp3_player"
 				(path "/0f0043d3-9467-400d-886a-57a73f910f34/4f719e08-a5fd-46cb-a375-4f681db4c0e1"
-					(reference "#PWR034")
+					(reference "#PWR037")
 					(unit 1)
 				)
 				(path "/0f0043d3-9467-400d-886a-57a73f910f34/cfa83fee-df6a-42e6-9021-3f2792ba73ef"
-					(reference "#PWR041")
+					(reference "#PWR031")
 					(unit 1)
 				)
@@
 		(dnp no)
 		(fields_autoplaced yes)
-		(property "Reference" "L5"
+		(property "Reference" "L1"
 			(at 69.85 26.67 0)
 			(show_name no)
@@
 				)
 				(path "/0f0043d3-9467-400d-886a-57a73f910f34/cfa83fee-df6a-42e6-9021-3f2792ba73ef"
-					(reference "L5")
+					(reference "L1")
 					(unit 1)
 				)
@@
 		(dnp no)
 		(fields_autoplaced yes)
-		(property "Reference" "#PWR039"
+		(property "Reference" "#PWR029"
 			(at 49.53 62.23 0)
 			(hide yes)
@@
 			(project "mp3_player"
 				(path "/0f0043d3-9467-400d-886a-57a73f910f34/4f719e08-a5fd-46cb-a375-4f681db4c0e1"
-					(reference "#PWR032")
+					(reference "#PWR035")
 					(unit 1)
 				)
 				(path "/0f0043d3-9467-400d-886a-57a73f910f34/cfa83fee-df6a-42e6-9021-3f2792ba73ef"
-					(reference "#PWR039")
+					(reference "#PWR029")
 					(unit 1)
 				)
@@
 		(dnp no)
 		(fields_autoplaced yes)
-		(property "Reference" "#PWR042"
+		(property "Reference" "#PWR032"
 			(at 86.36 62.23 0)
 			(hide yes)
@@
 			(project "mp3_player"
 				(path "/0f0043d3-9467-400d-886a-57a73f910f34/4f719e08-a5fd-46cb-a375-4f681db4c0e1"
-					(reference "#PWR035")
+					(reference "#PWR038")
 					(unit 1)
 				)
 				(path "/0f0043d3-9467-400d-886a-57a73f910f34/cfa83fee-df6a-42e6-9021-3f2792ba73ef"
-					(reference "#PWR042")
+					(reference "#PWR032")
 					(unit 1)
 				)
@@
 		(dnp no)
 		(fields_autoplaced yes)
-		(property "Reference" "C15"
+		(property "Reference" "C7"
 			(at 36.83 21.5962 0)
 			(show_name no)
@@
 				)
 				(path "/0f0043d3-9467-400d-886a-57a73f910f34/cfa83fee-df6a-42e6-9021-3f2792ba73ef"
-					(reference "C15")
+					(reference "C7")
 					(unit 1)
 				)
@@
 		(dnp no)
 		(fields_autoplaced yes)
-		(property "Reference" "#PWR040"
+		(property "Reference" "#PWR030"
 			(at 54.61 62.23 0)
 			(hide yes)
@@
 			(project "mp3_player"
 				(path "/0f0043d3-9467-400d-886a-57a73f910f34/4f719e08-a5fd-46cb-a375-4f681db4c0e1"
-					(reference "#PWR033")
+					(reference "#PWR036")
 					(unit 1)
 				)
 				(path "/0f0043d3-9467-400d-886a-57a73f910f34/cfa83fee-df6a-42e6-9021-3f2792ba73ef"
-					(reference "#PWR040")
+					(reference "#PWR030")
 					(unit 1)
 				)
@@
 		(in_pos_files yes)
 		(dnp no)
-		(property "Reference" "R18"
+		(property "Reference" "R16"
 			(at 24.13 38.354 90)
 			(show_name no)
@@
 				)
 				(path "/0f0043d3-9467-400d-886a-57a73f910f34/cfa83fee-df6a-42e6-9021-3f2792ba73ef"
-					(reference "R18")
-					(unit 1)
-				)
+					(reference "R16")
+					(unit 1)
+				)
