File: kicad/mp3_player/mp3_player.kicad_pcb (KiCad board)
At the start: 2 copper layers, 30 parts, among them J1 Conn_USB_C_Socket, SW1 Boot, SW2 Reset, SW3 RotaryEncoder_Switch, U1 MPU6500-breakout, U2 HC-SR04_Ultrasonic_Sensor, U3 ESP32-S3-WROOM-1, U4 AHT20_BMP280, U5 AMS1117-3.3

Commit message: [UPDATE] the desing of the schematic to use the current audio module
Parts:
- added C10: 220pF_0603_25V, Capacitor_SMD:C_0603_1608Metric_Pad1.08x0.95mm_HandSolder, F.Cu at (223.8, 110.5)
- added C11: 10uF, PCM_SparkFun-Capacitor:C_1210_3225Metric, F.Cu at (32.4, 88.5)
- added C12: 0.1uF, PCM_SparkFun-Capacitor:C_0603_1608Metric, F.Cu at (41.6, 92.9)
- added C13: 220pF_0603_25V, Capacitor_SMD:C_01005_0402Metric_Pad0.57x0.30mm_HandSolder, F.Cu at (42.2, 87.2)
- added C14: 220pF_0603_25V, Capacitor_SMD:C_0603_1608Metric_Pad1.08x0.95mm_HandSolder, F.Cu at (37.4, 92.9)
- added C8: 0.1uF, PCM_SparkFun-Capacitor:C_0603_1608Metric, F.Cu at (227.9, 110.5)
- added C9: 220pF_0603_25V, Capacitor_SMD:C_01005_0402Metric_Pad0.57x0.30mm_HandSolder, F.Cu at (228.5, 104.8)
- added D1: WS2812B, PCM_SparkFun-LED:WS2812_2020, F.Cu at (159.4, 100.3)
- added J2: Conn_USB_C_Socket, PCM_fab:Conn_USB_C_Socket_Molex_2171790001, F.Cu at (20.0, 54.9)
- added L1: 33nH, PCM_Resistor_SMD_AKL:R_0603_1608Metric_Pad0.98x0.95mm_HandSolder, F.Cu at (218.1, 109.5)
- added L2: 33nH, PCM_Resistor_SMD_AKL:R_0603_1608Metric_Pad0.98x0.95mm_HandSolder, F.Cu at (218.1, 112.1)
- added L3: 33nH, PCM_Resistor_SMD_AKL:R_0603_1608Metric_Pad0.98x0.95mm_HandSolder, F.Cu at (31.8, 91.9)
- added L4: 33nH, PCM_Resistor_SMD_AKL:R_0603_1608Metric_Pad0.98x0.95mm_HandSolder, F.Cu at (31.8, 94.4)
- added R11: 1M, Resistor_THT:R_Axial_DIN0207_L6.3mm_D2.5mm_P10.16mm_Horizontal, F.Cu at (15.2, 71.4)
- added R12: 5.1k, Resistor_THT:R_Axial_DIN0207_L6.3mm_D2.5mm_P10.16mm_Horizontal, F.Cu at (28.2, 56.9)
- added R13: 5.1k, Resistor_THT:R_Axial_DIN0207_L6.3mm_D2.5mm_P10.16mm_Horizontal, F.Cu at (28.0, 63.4)
- added R14: 10k, Resistor_THT:R_Axial_DIN0207_L6.3mm_D2.5mm_P10.16mm_Horizontal, F.Cu at (71.6, 52.9)
- added R15: 10k, Resistor_THT:R_Axial_DIN0207_L6.3mm_D2.5mm_P10.16mm_Horizontal, F.Cu at (71.6, 57.9)
- added R16: 1M, Resistor_THT:R_Axial_DIN0207_L6.3mm_D2.5mm_P10.16mm_Horizontal, F.Cu at (217.5, 102.0)
- added R17: 1M, Resistor_THT:R_Axial_DIN0207_L6.3mm_D2.5mm_P10.16mm_Horizontal, F.Cu at (31.2, 84.4)
- added U6: MAX98357A, Package_DFN_QFN:TQFN-16-1EP_3x3mm_P0.5mm_EP1.23x1.23mm, F.Cu at (224.6, 106.7)
- added U7: MAX98357A, Package_DFN_QFN:TQFN-16-1EP_3x3mm_P0.5mm_EP1.23x1.23mm, F.Cu at (38.3, 89.0)
- C2: value 100nF_Ceramic -> 1nF_Ceramic
- C3: value 1nF_Ceramic -> 10uF
- C4, C6: value 10uF -> 100nF
- C5: value 100nF -> 10uF
- C7: value 100nF -> 10uF; footprint Capacitor_THT:C_Disc_D5.0mm_W2.5mm_P2.50mm -> PCM_SparkFun-Capacitor:C_1210_3225Metric
- J1: value Conn_USB_C_Socket -> microSD; footprint PCM_fab:Conn_USB_C_Socket_Molex_2171790001 -> PCM_SparkFun-Connector:microSD_External_Pin
- R10: value 10k -> R_0805; footprint Resistor_THT:R_Axial_DIN0207_L6.3mm_D2.5mm_P10.16mm_Horizontal -> PCM_Resistor_SMD_AKL:R_0805_2012Metric
- R5: value 220ohm -> R_0805; footprint Resistor_THT:R_Axial_DIN0207_L6.3mm_D2.5mm_P10.16mm_Horizontal -> PCM_Resistor_SMD_AKL:R_0805_2012Metric
- R6: value 1M -> R_0805; footprint Resistor_THT:R_Axial_DIN0207_L6.3mm_D2.5mm_P10.16mm_Horizontal -> PCM_Resistor_SMD_AKL:R_0805_2012Metric
- R7: value 5.1k -> R_0805; footprint Resistor_THT:R_Axial_DIN0207_L6.3mm_D2.5mm_P10.16mm_Horizontal -> PCM_Resistor_SMD_AKL:R_0805_2012Metric
- R8: value 5.1k -> 220ohm
- R9: value 10k -> R_1206; footprint Resistor_THT:R_Axial_DIN0207_L6.3mm_D2.5mm_P10.16mm_Horizontal -> PCM_Resistor_SMD_AKL:R_1206_3216Metric
- moved C2 207.1 mm to (17.2, 64.9)
- moved C7 159.5 mm to (218.8, 106.2)
- moved SW3 134.4 mm to (243.0, 28.0)
- moved C1 129.5 mm to (159.5, 93.0)
- moved R5 125.2 mm to (37.5, 99.0), turned to -90 degrees
- moved U2 118.4 mm to (51.3, 32.6), turned to 180 degrees
- moved U3 116.7 mm to (234.3, 75.0), turned to -90 degrees
- moved R8 111.8 mm to (142.3, 105.7)
- moved R9 95.7 mm to (160.3, 96.8)
- moved SW1 89.8 mm to (28.7, 43.4), turned to 90 degrees
- moved U4 82.1 mm to (80.7, 97.2)
- moved LCD1 76.3 mm to (215.5, 43.0)
- moved LED1 70.4 mm to (159.5, -60.0)
- moved U1 65.9 mm to (97.3, 97.1)
- moved C3 64.5 mm to (31.9, 50.4), turned to 0 degrees
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Connections:
- C1 pad 1: Net-(C1-Pad1) -> Net-(J1-CMD/SDI)
- C1 pad 2: Net-(U3-IO17) -> PWR_3V3
- C2 pad 1: Net-(U3-IO18) -> GND
- C2 pad 2: Net-(C2-Pad2) -> Net-(J2-SHIELD)
- C3 pad 1: GND -> 5V
- C3 pad 2: Net-(J1-SHIELD) -> Net-(U5-IN)
- C4 pad 1: 5V -> GND
- C4 pad 2: Net-(U5-IN) -> Net-(C4-Pad2)
- C5 pad 1: GND -> Net-(C4-Pad2)
- C5 pad 2: Net-(C5-Pad2) -> PWR_3V3
- C6 pad 1: Net-(C5-Pad2) -> Net-(U5-OUT)
- C7 pad 1: Net-(U5-OUT) -> GND
- C7 pad 2: PWR_3V3 -> 5V
- LS1 pad 1: Net-(C1-Pad1) -> /MAX98357/VD+
- LS1 pad 2: GND -> /MAX98357/VD-
- LS2 pad 1: Net-(C2-Pad2) -> /MAX98357/VD+
- LS2 pad 2: GND -> /MAX98357/VD-
- R10 pad 2: /ESP power/IO0 -> Net-(J1-DAT0/SDO)
- R5 pad 1: PWR_3V3 -> Net-(U3-IO40)
- R5 pad 2: Net-(LCD1-A) -> Net-(J1-DAT0/SDO)
- R6 pad 1: GND -> Net-(U3-IO39)
- R6 pad 2: Net-(J1-SHIELD) -> Net-(J1-CLK/SCK)
- R7 pad 1: Net-(J1-CC1) -> Net-(U3-IO38)
- R7 pad 2: GND -> Net-(J1-CMD/SDI)
- R8 pad 1: Net-(J1-CC2) -> PWR_3V3
- R8 pad 2: GND -> Net-(LCD1-A)
- R9 pad 2: /ESP power/EN -> Net-(J1-CMD/SDI)
- SW3 pad A: Net-(U3-IO16) -> Net-(U3-IO42)
- U3 pad 10: Net-(U3-IO17) -> /MAX98357/DIN
- U3 pad 11: Net-(U3-IO18) -> /MAX98357/DIN
- U3 pad 15: Net-(LED1-DIN) -> unconnected-(U3-IO3-Pad15)
- U3 pad 24: unconnected-(U3-IO47-Pad24) -> /MAX98357/LRCLK
- U3 pad 25: unconnected-(U3-IO48-Pad25) -> Net-(D1-DIN)
- U3 pad 31: unconnected-(U3-IO38-Pad31) -> Net-(U3-IO38)
- U3 pad 32: unconnected-(U3-IO39-Pad32) -> Net-(U3-IO39)
- U3 pad 33: unconnected-(U3-IO40-Pad33) -> Net-(U3-IO40)
- U3 pad 34: unconnected-(U3-IO41-Pad34) -> Net-(LED1-DIN)
- U3 pad 35: unconnected-(U3-IO42-Pad35) -> Net-(U3-IO42)
- U3 pad 9: Net-(U3-IO16) -> /MAX98357/BCLK
- U4 pad SCL: Net-(U1-EDA) -> Net-(U1-ECL)
- U4 pad SDA: Net-(U1-ECL) -> Net-(U1-EDA)
Routing:
- net GND: track 269.0 -> 0.00 mm
- net Net-(U1-ECL): track 181.2 -> 0.00 mm
- net Net-(U1-EDA): track 168.0 -> 0.00 mm
- net PWR_3V3: track 152.9 -> 0.00 mm
- net 5V: track 150.7 -> 0.00 mm
- net /ESP power/ESP32_USB_D-: track 138.9 -> 0.00 mm
- net /ESP power/ESP32_USB_D+: track 97.7 -> 0.00 mm
- net Net-(U3-IO17): track 46.9 -> 0.00 mm
- net Net-(U1-INT): track 31.9 -> 0.00 mm
- net Net-(LCD1-IC_S0): track 31.6 -> 0.00 mm
- net Net-(U3-IO0): track 30.7 -> 0.00 mm
- net Net-(LCD1-IC_CS): track 29.5 -> 0.00 mm
- net Net-(J1-SHIELD): track 26.8 -> 0.00 mm
- net Net-(LCD1-IC_S1): track 26.3 -> 0.00 mm
- net Net-(U5-OUT): track 11.0 -> 0.00 mm
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
Commit message: [ADD] lcd segment displays to the project
Parts:
- added C15: 0.1uF, Capacitor_THT:C_Rect_L31.5mm_W11.0mm_P27.50mm_MKS4, F.Cu at (232.3, 28.8)
- added C16: 0.1uF, Capacitor_THT:C_Rect_L31.5mm_W11.0mm_P27.50mm_MKS4, F.Cu at (232.3, 71.7)
- added D2: Blue, PCM_SparkFun-LED:LED_1206_3216Metric_Blue, F.Cu at (245.7, 60.6)
- added D3: Blue, PCM_SparkFun-LED:LED_1206_3216Metric_Blue, F.Cu at (245.7, 103.5)
- added DS1: WC2004A, Display:WC1602A, F.Cu at (32.1, 110.0)
- added DS2: WC1602A, Display:WC1602A, F.Cu at (32.1, 147.8)
- added J3: Conn_01x04, PCM_4ms_Connector:Pins_1x04_3.96mm_TH_MTA156, F.Cu at (218.3, 84.5)
- added J4: Conn_USB_C_Socket, PCM_fab:Conn_USB_C_Socket_Molex_2171790001, F.Cu at (235.3, 129.9)
- added POT1: 16mm_CtrDet_10k, PCM_Potentiometer_THT_AKL:Potentiometer_TT_P0915N, F.Cu at (258.2, 48.2)
- added POT2: 16mm_CtrDet_10k, PCM_Potentiometer_THT_AKL:Potentiometer_TT_P0915N, F.Cu at (258.2, 91.1)
- added Q1: S8050, Package_TO_SOT_THT:TO-92_Inline, F.Cu at (244.9, 56.5)
- added Q2: S8050, Package_TO_SOT_THT:TO-92_Inline, F.Cu at (244.9, 99.4)
- added R18: 1k, Resistor_THT:R_Axial_DIN0207_L6.3mm_D2.5mm_P10.16mm_Horizontal, F.Cu at (231.1, 37.1)
- added R19: 1k, Resistor_THT:R_Axial_DIN0207_L6.3mm_D2.5mm_P10.16mm_Horizontal, F.Cu at (231.1, 41.1)
- added R20: 1k, Resistor_THT:R_Axial_DIN0207_L6.3mm_D2.5mm_P10.16mm_Horizontal, F.Cu at (231.1, 45.2)
- added R21: 47k, Resistor_THT:R_Axial_DIN0207_L6.3mm_D2.5mm_P10.16mm_Horizontal, F.Cu at (231.1, 49.2)
- added R22: 1k, Resistor_THT:R_Axial_DIN0207_L6.3mm_D2.5mm_P10.16mm_Horizontal, F.Cu at (231.1, 53.3)
- added R23: 47k, Resistor_THT:R_Axial_DIN0207_L6.3mm_D2.5mm_P10.16mm_Horizontal, F.Cu at (231.1, 57.3)
- added R24: 47k, Resistor_THT:R_Axial_DIN0207_L6.3mm_D2.5mm_P10.16mm_Horizontal, F.Cu at (231.1, 61.4)
- added R25: 1k, Resistor_THT:R_Axial_DIN0207_L6.3mm_D2.5mm_P10.16mm_Horizontal, F.Cu at (231.1, 80.0)
- added R26: 1k, Resistor_THT:R_Axial_DIN0207_L6.3mm_D2.5mm_P10.16mm_Horizontal, F.Cu at (231.1, 84.0)
- added R27: 1k, Resistor_THT:R_Axial_DIN0207_L6.3mm_D2.5mm_P10.16mm_Horizontal, F.Cu at (231.1, 88.1)
- added R28: 47k, Resistor_THT:R_Axial_DIN0207_L6.3mm_D2.5mm_P10.16mm_Horizontal, F.Cu at (231.1, 92.1)
- added R29: 1k, Resistor_THT:R_Axial_DIN0207_L6.3mm_D2.5mm_P10.16mm_Horizontal, F.Cu at (231.1, 96.2)
- added R30: 47k, Resistor_THT:R_Axial_DIN0207_L6.3mm_D2.5mm_P10.16mm_Horizontal, F.Cu at (231.1, 100.2)
- added R31: 47k, Resistor_THT:R_Axial_DIN0207_L6.3mm_D2.5mm_P10.16mm_Horizontal, F.Cu at (231.1, 104.3)
- added TP1: TestPoint_2Pole, Connector_PinHeader_2.00mm:PinHeader_1x02_P2.00mm_Horizontal, F.Cu at (244.9, 37.1)
- added TP2: TestPoint_2Pole, Connector_PinHeader_2.00mm:PinHeader_1x02_P2.00mm_Horizontal, F.Cu at (244.9, 43.1)
- added TP3: TestPoint_2Pole, Connector_PinHeader_2.00mm:PinHeader_1x02_P2.00mm_Horizontal, F.Cu at (244.9, 49.2)
- added TP4: TestPoint_2Pole, Connector_PinHeader_2.00mm:PinHeader_1x02_P2.00mm_Horizontal, F.Cu at (244.9, 80.0)
- added TP5: TestPoint_2Pole, Connector_PinHeader_2.00mm:PinHeader_1x02_P2.00mm_Horizontal, F.Cu at (244.9, 86.0)
- added TP6: TestPoint_2Pole, Connector_PinHeader_2.00mm:PinHeader_1x02_P2.00mm_Horizontal, F.Cu at (244.9, 92.1)
- added U8: PCF8574T, Package_SO:SOIC-16W_7.5x10.3mm_P1.27mm, F.Cu at (259.6, 55.9)
- added U9: PCF8574T, Package_SO:SOIC-16W_7.5x10.3mm_P1.27mm, F.Cu at (259.6, 98.8)
- J2: value Conn_USB_C_Socket -> Conn_01x04; footprint PCM_fab:Conn_USB_C_Socket_Molex_2171790001 -> PCM_4ms_Connector:Pins_1x04_3.96mm_TH_MTA156
- moved C2 232.2 mm to (244.9, 110.3)
- moved C11 224.8 mm to (255.7, 114.5)
- moved C12 224.8 mm to (264.9, 118.9)
- moved C13 224.8 mm to (265.5, 113.2)
- moved C14 224.8 mm to (260.7, 118.9)
- moved L3 224.8 mm to (255.1, 117.9)
- moved L4 224.8 mm to (255.1, 120.4)
- moved R17 224.8 mm to (254.4, 110.3)
- moved U7 224.8 mm to (261.5, 115.0)
- moved C3 222.4 mm to (244.9, 114.4)
- moved R11 219.4 mm to (231.1, 110.3)
- moved U5 214.5 mm to (245.9, 132.7)
- moved J1 212.8 mm to (218.6, 34.5), turned to 0 degrees
- moved C6 211.7 mm to (244.9, 126.5)
- moved R12 210.9 mm to (231.1, 114.4)
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Connections:
- C10 pad 1: /MAX98357/VD- -> /MAX98358/VD-
- C2 pad 2: Net-(J2-SHIELD) -> Net-(J4-SHIELD)
- C9 pad 1: /MAX98357/VD+ -> /MAX98358/VD+
- L1 pad 2: /MAX98357/VD+ -> /MAX98358/VD+
- L2 pad 2: /MAX98357/VD- -> /MAX98358/VD-
- LS1 pad 1: /MAX98357/VD+ -> /MAX98358/VD+
- LS1 pad 2: /MAX98357/VD- -> /MAX98358/VD-
- R11 pad 2: Net-(J2-SHIELD) -> Net-(J4-SHIELD)
- R12 pad 1: Net-(J2-CC1) -> Net-(J4-CC1)
- R13 pad 1: Net-(J2-CC2) -> Net-(J4-CC2)
- R3 pad 1: Net-(U1-ECL) -> /I2C/SCL
- R4 pad 1: Net-(U1-EDA) -> /I2C/SDA
- SW3 pad C: unconnected-(SW3-PadC) -> GND
- U1 pad 3: Net-(U1-ECL) -> /I2C/SCL
- U1 pad 4: Net-(U1-EDA) -> /I2C/SDA
- U1 pad 5: Net-(U1-EDA) -> /I2C/SDA
- U1 pad 6: Net-(U1-ECL) -> /I2C/SCL
- U3 pad 10: /MAX98357/DIN -> /MAX98358/DIN
- U3 pad 38: Net-(U1-EDA) -> /I2C/SDA
- U3 pad 39: Net-(U1-ECL) -> /I2C/SCL
- U4 pad SCL: Net-(U1-ECL) -> /I2C/SCL
- U4 pad SDA: Net-(U1-EDA) -> /I2C/SDA
- U6 pad 1: /MAX98357/DIN -> /MAX98358/DIN
- U6 pad 2: /MAX98357/GAIN -> /MAX98358/GAIN
