File: kicad/mp3_player/onboard_i2c.kicad_sch (KiCad schematic)
At the start: 15 parts, among them Q1 S8050, U8 PCF8574T

Commit message: [UPDATE] the KiCad schematic to show the pins requiring bridging on the I2C
Connections:
- net A0 renamed A0(1)
- net A1 renamed A1(1)
- net A2 renamed A2(1)
- net GND renamed A0(2)
Changed lines of the file:
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@@
+		)
+	)
+	(hierarchical_label "A2(2)"
+		(shape input)
+		(at 36.83 71.12 270)
+		(effects
+			(font
+				(size 1.27 1.27)
+			)
+			(justify right)
+		)
+	)
+	(hierarchical_label "A2(1)"
+		(shape input)
+		(at 36.83 49.53 90)
+		(effects
+			(font
+				(size 1.27 1.27)
+			)
+			(justify left)
 		)
 	)
@@
 		)
 	)
+	(hierarchical_label "A0(1)"
+		(shape input)
+		(at 20.32 49.53 90)
+		(effects
+			(font
+				(size 1.27 1.27)
+			)
+			(justify left)
+		)
+	)
 	(hierarchical_label "E"
 		(shape input)
@@
 		)
 	)
+	(hierarchical_label "A1(1)"
+		(shape input)
+		(at 27.94 49.53 90)
+		(effects
+			(font
+				(size 1.27 1.27)
+			)
+			(justify left)
+		)
+	)
 	(hierarchical_label "V0"
 		(shape input)
@@
 		)
 	)
+	(hierarchical_label "A0(2)"
+		(shape input)
+		(at 20.32 71.12 270)
+		(effects
+			(font
+				(size 1.27 1.27)
+			)
+			(justify right)
+		)
+	)
 	(hierarchical_label "(K) BL-"
 		(shape input)
@@
 		(effects
 			(font
+				(size 1.27 1.27)
+			)
+			(justify right)
+		)
+	)
+	(hierarchical_label "A1(2)"
+		(shape input)
+		(at 27.94 73.66 270)
+		(effects
+			(font
